Commit message: sim: joint effort limits 10 -> 3 N.m to match the real STS3215
The URDF/MJCF carried a 10 N.m effort limit on all 7 joints, well above what
an STS3215 actually delivers. The gap let policies learn torques the real arm
cannot produce, which showed up as the arm stalling mid-lift on hardware.

File: simulation/urdf/components/so101_arm/so101_new_calib.urdf (robot description, URDF)
Before this commit: robot so101_new_calib, 8 links, 7 joints
Joints:
- joint elbow_flex: limit lower=-1.69 upper=1.69 effort=10 velocity=10 -> lower=-1.69 upper=1.69 effort=3 velocity=10
- joint gripper: limit lower=-0.174533 upper=1.74533 effort=10 velocity=10 -> lower=-0.174533 upper=1.74533 effort=3 velocity=10
- joint shoulder_lift: limit lower=-1.74533 upper=1.74533 effort=10 velocity=10 -> lower=-1.74533 upper=1.74533 effort=3 velocity=10
- joint shoulder_pan: limit lower=-1.91986 upper=1.91986 effort=10 velocity=10 -> lower=-1.91986 upper=1.91986 effort=3 velocity=10
- joint wrist_flex: limit lower=-1.65806 upper=1.65806 effort=10 velocity=10 -> lower=-1.65806 upper=1.65806 effort=3 velocity=10
- joint wrist_roll: limit lower=-2.74385 upper=2.84121 effort=10 velocity=10 -> lower=-2.74385 upper=2.84121 effort=3 velocity=10

File: simulation/urdf/so101_on_frame.urdf (robot description, URDF)
Before this commit: robot so101_on_frame, 67 links, 66 joints
Links:
- link 100cm_4: geometry collision box size=0.02 0.02 1.0; visual mesh filename=components/base_frame/meshes/_100cm.stl scale=1 1 1
Joints:
- joint elbow_flex: limit lower=-1.69 upper=1.69 effort=10 velocity=10 -> lower=-1.69 upper=1.69 effort=3 velocity=10
- joint gripper: limit lower=-0.174533 upper=1.74533 effort=10 velocity=10 -> lower=-0.174533 upper=1.74533 effort=3 velocity=10
- joint shoulder_lift: limit lower=-1.74533 upper=1.74533 effort=10 velocity=10 -> lower=-1.74533 upper=1.74533 effort=3 velocity=10
- joint shoulder_pan: limit lower=-1.91986 upper=1.91986 effort=10 velocity=10 -> lower=-1.91986 upper=1.91986 effort=3 velocity=10
- joint wrist_flex: limit lower=-1.65806 upper=1.65806 effort=10 velocity=10 -> lower=-1.65806 upper=1.65806 effort=3 velocity=10
- joint wrist_roll: limit lower=-2.74385 upper=2.84121 effort=10 velocity=10 -> lower=-2.74385 upper=2.84121 effort=3 velocity=10
