Commit message: Add MuJoCo (MJCF) model with 2 cameras; simulation README with renders; rename frame_camera_wrist -> frame_wrist_camera

File: simulation/urdf/so101_on_frame.urdf (robot description, URDF)
Before this commit: robot so101_on_frame, 67 links, 66 joints
Links:
- removed link frame_camera_wrist
- added link frame_wrist_camera, mass 1e-6
Joints:
- removed joint frame_camera_wrist_joint
- added joint frame_wrist_camera_joint: type fixed, parent gripper_link, child frame_wrist_camera, origin xyz=0.0025 0.0675 -0.0062 rpy=-2.7071 0 3.14159

Commit message: RL: add rl/maniskill (vision-based Squint policy) alongside rl/mjlab
Splits the RL work into two implementations of the same pick-and-place
task: rl/mjlab (state-based, existing) and rl/maniskill (new, vision-only,
built on ManiSkill3 + Squint). Key pieces:

- SO-101-on-frame ManiSkill agent with the rail slider as a 7th DOF and
  dual wrist/overhead cameras, calibrated from the shared URDF.
- Fixed a real SAPIEN-vs-MuJoCo camera convention mismatch in the URDF
  (both camera joints had roll off by pi for SAPIEN's rendering
  convention), and added real collision to the lightbox panels (URDF and
  MJCF) so objects don't fall through.
- Pick-and-place task with cube/bin spawning in separate regions along
  the rail's travel axis, so solving it actually requires sliding.
- Reshaped reward (raised the success bonus and gated the "static robot"
  bonus on actually releasing the item) after training found a "hold the
  cube near the goal forever" exploit that nearly matched the success
  reward.
- realism_mode: ray-traced shading, real PBR textures, and an overhead
  softbox area light for one-off high-fidelity renders (never used
  during training).
- USD import pipeline (simulation/usd/import_mjcf.py) that generates a
  physics-enabled Isaac Lab asset from the MJCF via Isaac Sim's own MJCF
  importer, instead of hand-authoring UsdPhysics schemas.

Trained checkpoint (slider_pickplace_v7, 5M steps) reaches ~62-81%
success across eval checkpoints; shipped separately in a prior commit.

File: simulation/urdf/so101_on_frame.urdf (robot description, URDF)
Before this commit: robot so101_on_frame, 67 links, 66 joints
Links:
- link part_1: geometry collision box size=1.04 0.54 0.002; visual mesh filename=components/base_frame/meshes/Part_1.stl scale=1 1 1
- link part_1_1: geometry collision box size=1.04 0.51 0.002; visual mesh filename=components/base_frame/meshes/Part_1_1.stl scale=1 1 1
- link part_1_2: geometry collision box size=0.51 0.54 0.002; visual mesh filename=components/base_frame/meshes/Part_1_2.stl scale=1 1 1
- link part_1_3: geometry collision box size=0.51 0.54 0.002; visual mesh filename=components/base_frame/meshes/Part_1_2.stl scale=1 1 1
Joints:
- joint fix_1: origin xyz=-3.46945e-18 0 0 rpy=-1.5708 -0 3.14159 -> xyz=-3.46945e-18 0 0.01 rpy=-1.5708 -0 3.14159
- joint frame_overhead_camera: origin xyz=-0.006 0.0339256 -0.0752492 rpy=-2.53073 -0 0 -> xyz=-0.006 0.0339256 -0.0752492 rpy=0.0 0.959929 1.570778
- joint frame_wrist_camera_joint: origin xyz=0.0025 0.0675 -0.0062 rpy=-2.7071 0 3.14159 -> xyz=0.0025 0.0675 -0.0062 rpy=0.0 1.136305 -1.570797

Commit message: URDF: roll wrist camera 180 deg about its optical axis (upside-down mount)
The physical wrist camera sits upside down in its holder, so its image
arrives rotated 180 degrees; baking the pi roll into the camera joint
reproduces exactly that image rotation with no other geometric change
and no per-frame image processing. Also keep render_chained_eval's
cameras steady (zero pose/fov jitter) even when rendering with domain
randomization on -- in a video the jitter just reads as shake.

File: simulation/urdf/so101_on_frame.urdf (robot description, URDF)
Before this commit: robot so101_on_frame, 67 links, 66 joints
Joints:
- joint frame_wrist_camera_joint: origin xyz=0.0025 0.0675 -0.0062 rpy=0.0 1.136305 -1.570797 -> xyz=0.0025 0.0675 -0.0062 rpy=3.141593 1.136305 -1.570797

Commit message: Simulation: split fixed-jaw collision so the gripper grips flush
A single convex hull of the concave fixed-jaw mesh stands ~7 mm proud
of the true surface at the finger (2.6x the mesh volume), so objects
were gripped with ~1 cm of visible daylight. Splitting the collision
into a base piece and a finger piece (geometry from Squint's
so101.urdf, github.com/aalmuzairee/squint, shipped as each piece's
convex hull) drops the finger's standoff to ~2.5 mm mean / 4.8 mm p90.

Applied to the URDF and MJCF, and the Isaac USD asset regenerated from
the MJCF via simulation/usd/import_mjcf.py (drop-test validated at the
documented physics_dt=1/500).

File: simulation/urdf/so101_on_frame.urdf (robot description, URDF)
Before this commit: robot so101_on_frame, 67 links, 66 joints
Links:
- link gripper_link: geometry collision mesh filename=components/so101_arm/assets/fixed_jaw_base_convex.obj; collision mesh filename=components/so101_arm/assets/fixed_jaw_finger_convex.obj

Commit message: mjlab: real-speed rate limit in the action space, 3 N.m effort, no penalties
Three coupled fixes, because the missing rate limit is why the penalties existed.

1. Action space was not a delta. JointPositionActionCfg(use_default_offset=True)
   gives target = action * scale + default_joint_pos: an ABSOLUTE target measured
   from home. Nothing bounded per-step motion -- one step could command the full
   +-scale swing from home, consecutive steps the whole 2*scale range. The config
   comment called it "delta joint position", which it never was. Switched to
   RelativeJointPositionActionCfg (target = current_pos + action * scale), so
   scale is a hard per-step cap.

2. Action scale now comes from measured real speed, not from torque. It was
   mjlab's yam heuristic, 0.25 * effort_limit / stiffness, which ties step size
   to torque through a relationship with no physical meaning -- it gave the arm
   0.14 rad/step, ~7 rad/s at 50 Hz, 14x the real servo. Now
   real_speed / CONTROL_HZ from the measured rig (arm 0.5 rad/s, rail 7 cm/s,
   gripper 2.0 rad/s), which lands exactly on the maniskill twin's numbers:
   0.05 rad/step, 0.007 m/step, 0.2 rad/step.

3. Effort limits 10 -> 3 N.m. get_spec() deletes the XML actuators, discarding
   the forcerange="-3.0 3.0" that sts3215.xml already had correct, and
   BuiltinPositionActuatorCfg re-declared them at 10.

Then the penalties come out, since they were standing in for (1):
action_rate_l2, joint_vel_hinge, and the joint_vel_hinge_weight ramp curriculum.
joint_vel_hinge's max_vel was 0.5 -- literally the real arm's 0.5 rad/s -- so it
was a soft reward-level approximation of the hard cap. Its own comment made the
case against it: the weight had to be ramped linearly or it "can collapse a
trained policy", and had to stay under ~-0.06 or "carrying stops paying". A cap
in the action space has no weight and no window to fall out of.

Also fixed, found on the way:
- decimation 4 -> 20, i.e. 50 Hz -> 10 Hz control, matching the maniskill twin
  and the deploy loop's 10 Hz portal tick. Control cadence is part of the
  sim2real contract. episode_length_s 10 -> 30 keeps the 300-step horizon.
- the rail's actuatorfrcrange was -1 1 (N, prismatic). MuJoCo applies the joint
  clamp on top of the actuator's forcerange, so 1 N capped the rail no matter
  what the actuator said -- not enough to accelerate the gantry + arm. Now 100 N,
  matching what maniskill drives it at. Same for the URDF's effort="1"; maniskill
  overrode it with force_limit=100 so it never bit there, but the model should
  not carry a value the rig contradicts.

Verified:
- config builds: RelativeJointPositionActionCfg, per-joint scale as above,
  decimation 20 -> 10.0 Hz, 300-step episodes, rewards down to 5 task terms +
  joint_pos_limits, curriculum down to placement_spread
- MJCF loads: all six arm joints and their actuators at +-3, rail at +-100
- maniskill unaffected by the shared URDF edit: force limits still 3 N.m on the
  arm and 100 N on the rail, rail still tracking 0.0067 of its 0.007 m/step cap

NOT addressed: RelativeJointPositionAction is delta-from-CURRENT-position, while
maniskill uses pd_joint_target_delta_pos (delta from the previous TARGET) and
deploy integrates into a running target the same way. Delta-from-current stalls
when a joint lags, since the target can never lead the measured pose; the other
two cannot. mjlab has no delta-from-target term, so this is a real remaining
divergence between the stacks.

File: simulation/urdf/so101_on_frame.urdf (robot description, URDF)
Before this commit: robot so101_on_frame, 67 links, 66 joints
Joints:
- joint dof_slider: limit lower=-0.40286 upper=0.41714 effort=1 velocity=1 -> lower=-0.40286 upper=0.41714 effort=100 velocity=1

Commit message: assets: drop the frame handles and the M5 screws from the visual geometry
The render stage is entirely geometry-bound -- at 512 envs, rendering at 32 px instead of
128 px changes the step by 1.3% -- so the visual triangle budget IS the render cost. It was
756k triangles per env, and two of the biggest line items are hardware no camera needs:

  Handle.stl                  49,380 tris x2 = 98,760  (13.1%)
  M5x25_low_profile_screw.stl  6,062 tris x4 =  24,248  ( 3.2%)

633k now, 16.3% off. Frame carry handles and four gantry screws, at rail height half a
metre above the work surface.

Only the <visual> blocks go. The links and their fixed joints stay, because two of the screw
links carry other hardware beneath them (m5x25_low_profile_screw_2 -> a wheel spacer,
_3 -> a nylock) and re-parenting those needs origin composition. That leaves six links with
neither visual nor collision, which is a physics-side concern rather than a render one: the
articulation still has 67 links of which only 12 carry collision, and collapsing all of the
visual-only fixed links is a separate job.

Collision geometry is untouched -- these meshes were never referenced by a <collision>.

File: simulation/urdf/so101_on_frame.urdf (robot description, URDF)
Before this commit: robot so101_on_frame, 67 links, 66 joints
Links:
- link handle: geometry 
- link handle_1: geometry 
- link m5x25_low_profile_screw: geometry 
- link m5x25_low_profile_screw_1: geometry 
- link m5x25_low_profile_screw_2: geometry 
- link m5x25_low_profile_screw_3: geometry 

Commit message: assets: drop the rail drive internals, keep its enclosure
The rail drive assembly is one chain off root, all of it within a few cm at z~0.51 m (rail
height, half a metre above the work surface):

  root -> sg_ziji_15 -> xg_ziji_16 -> motor_1723_3 -> pcb_chazuo_92 -> ge_27
       -> metal servo horn (drive) -> pinion,  plus zk_122 -> horn (driven)

Removed the internals, kept the three enclosure/bracket parts:

  GE_27              42,444   an 18 mm cube carrying 42k triangles, the worst
  MOTOR_1723_3        9,100   ratio in the whole rig
  Pinion              8,336
  metal horn (drive)  3,000
  metal horn (driven) 2,148
  PCB_CHAZUO_92         948
                     ------
                     65,976

  kept: SG_ZIJI_15 19,032, XG_ZIJI_16 16,170, ZK_122 4,286

567k triangles per env now, 25% off the original 756k across handles, screws and this.

Visual blocks only again, so the kinematic chain through the drive is intact -- the removed
links stay as frames because the enclosure parts hang off them.

File: simulation/urdf/so101_on_frame.urdf (robot description, URDF)
Before this commit: robot so101_on_frame, 67 links, 66 joints
Links:
- link ge_27: geometry 
- link motor_1723_3: geometry 
- link pcb_chazuo_92: geometry 
- link pinion: geometry 
- link 金属舵盘_从动__v2: geometry 
- link 金属舵盘_驱动__v2: geometry 
